File: Design/eagle/driver.sch (EAGLE design)
At the start: 44 parts, among them IC1 V_REG_LD1117VXX, Q1 600mA/40V, Q10 600mA/40V, Q11 600mA/40V, Q13 600mA/40V, Q14 600mA/40V, Q15 600mA/40V, Q2 600mA/40V, Q3 600mA/40V, Q5 600mA/40V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

Commit message: Agregadas correcciones en PCB
Parts:
- C1: value 1mF -> 1000uF
- C2: value 1.0uF -> 10uF
Changed lines of the file:
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@@
 <part name="SUPPLY28" library="SparkFun-PowerSymbols" deviceset="VCC" device=""/>
 <part name="M2" library="SparkFun-Connectors" deviceset="CONN_02" device="3.5MM"/>
-<part name="C1" library="SparkFun-Capacitors" deviceset="1000UF" device="-RADIAL-5MM-25V-20%" value="1mF"/>
+<part name="C1" library="SparkFun-Capacitors" deviceset="1000UF" device="-RADIAL-5MM-25V-20%" value="1000uF"/>
 <part name="SUPPLY29" library="supply2" deviceset="GND" device=""/>
-<part name="C2" library="SparkFun-Capacitors" deviceset="1.0UF" device="-0805-25V-10%" value="1.0uF"/>
+<part name="C2" library="SparkFun-Capacitors" deviceset="1.0UF" device="-0805-25V-10%" value="10uF"/>
 <part name="S1" library="SparkFun-Switches" deviceset="SWITCH-SPDT" device="-PTH-11.6X4.0MM"/>
 <part name="M3" library="SparkFun-Connectors" deviceset="CONN_02" device="3.5MM"/>
